File: arm-adaptor.brd (EAGLE design)
At the start: 10 parts, among them IC2 ATMEGA644-20PU, X1 MICROSD

Commit message: Design for Arduino DUE shield -> Sanguinololu.
Routing:
- net GND: track 65.1 -> 68.3 mm, vias 13 -> 12
Changed lines of the file:
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@@
 <?xml version="1.0" encoding="utf-8"?>
 <!DOCTYPE eagle SYSTEM "eagle.dtd">
-<eagle version="6.2">
+<eagle version="6.3">
 <drawing>
 <settings>
@@
 </class>
 </classes>
-<designrules>
+<designrules name="default">
 <description language="de">&lt;b&gt;EAGLE Design Rules&lt;/b&gt;
 &lt;p&gt;
@@
 <wire x1="78.945" y1="21.355" x2="79.0575" y2="21.355" width="0.4064" layer="1"/>
 <via x="57.785" y="10.16" extent="1-16" drill="0.6" diameter="2.1844"/>
-<wire x1="57.785" y1="10.16" x2="66.04" y2="10.16" width="0.4064" layer="16"/>
-<via x="66.04" y="10.16" extent="1-16" drill="0.6" diameter="2.1844"/>
-<via x="68.8975" y="10.16" extent="1-16" drill="0.6" diameter="2.1844"/>
-<wire x1="68.8975" y1="10.16" x2="76.2" y2="10.16" width="0.4064" layer="16"/>
+<wire x1="57.785" y1="10.16" x2="67.6275" y2="10.16" width="0.4064" layer="16"/>
+<via x="67.6275" y="10.16" extent="1-16" drill="0.6" diameter="2.1844"/>
+<wire x1="68.8975" y1="10.16" x2="68.8975" y2="10.16" width="0" layer="19" extent="1-16"/>
+<wire x1="68.8975" y1="10.16" x2="69.215" y2="10.16" width="0" layer="19" extent="1-16"/>
 <via x="76.2" y="10.16" extent="1-16" drill="0.6" diameter="2.1844"/>
+<wire x1="67.6275" y1="10.16" x2="76.2" y2="10.16" width="0.4064" layer="16"/>
 <wire x1="76.445" y1="24.455" x2="79.0575" y2="24.455" width="0.4064" layer="1"/>
 <wire x1="79.0575" y1="24.455" x2="79.0575" y2="24.4475" width="0.4064" layer="1"/>
 <wire x1="79.0575" y1="24.4475" x2="78.945" y2="24.4475" width="0.4064" layer="1"/>
 <wire x1="78.945" y1="24.4475" x2="78.945" y2="21.355" width="0.4064" layer="1"/>
+<wire x1="69.215" y1="10.16" x2="67.6275" y2="10.16" width="0" layer="19" extent="1-16"/>
+<wire x1="67.6275" y1="10.16" x2="67.6275" y2="9.8425" width="0.4064" layer="16"/>
 </signal>
 <signal name="PB7-SCK">
